File: hw/sch_pcb/ISO11446PWR01.kicad_pcb (KiCad board)
At the start: 2 copper layers, 40.1 x 40.1 mm, 8 parts, among them J1 Umin ... Umax, M1 HOLE M3, M2 HOLE M3, M3 HOLE, M4 HOLE

Commit message: testing schema
Parts:
- added F1: Fuse, Fuse:Fuse_Bourns_MF-RG400, F.Cu at (199.5, 84.2)
- added F2: Polyfuse, Fuse:Fuse_Bourns_MF-RG400, F.Cu at (213.4, 94.0)
- added J1: HEADER_2x04_PARALLEL, Mlab_Pin_Headers:Straight_2x04, F.Cu at (243.8, 55.9)
- added J2: HEADER_2x04_PARALLEL, Mlab_Pin_Headers:Straight_2x04, F.Cu at (262.9, 102.9)
- added J3: HEADER_2x04_PARALLEL, Mlab_Pin_Headers:Straight_2x04, F.Cu at (248.9, 76.2)
- added J4: Conn_01x01_Female, Mlab_CON:WAGO256, F.Cu at (215.9, 114.3)
- added J5: Conn_01x01_Female, Mlab_CON:WAGO256, F.Cu at (228.6, 55.9)
- added J6: Conn_01x01_Female, Mlab_CON:WAGO256, F.Cu at (215.9, 43.2)
- added J7: Conn_01x01_Female, Mlab_CON:WAGO256, F.Cu at (215.9, 119.4)
- renumbered J1 to J8
Connections:
- M1 pad 1: GND -> Net-(M1-Pad1)
- M2 pad 1: GND -> Net-(M1-Pad1)
- M3 pad 1: GND -> Net-(M1-Pad1)
- M4 pad 1: GND -> Net-(M1-Pad1)
