File: hw/sch_pcb/ISO11446PWR01.kicad_pcb (KiCad board)
At the start: 2 copper layers, 70.6 x 90.9 mm, 70 parts, among them J1 WAGO 256-401, J10 WAGO 256-401, J11 WAGO 256-401, J13 WAGO 256-401, J14 3.3-5V, J15 Signals, J16 2x4, J18 2x4, J19 WAGO 256-401, J2 WAGO 256-401, J20 WAGO 256-401, J21 WAGO 256-401, J22 WAGO 256-401, J3 WAGO 256-401, J4 WAGO 256-401, J5 WAGO 256-401, J6 WAGO 256-401, J7 WAGO 256-401, J8 WAGO 256-401, J9 WAGO 256-401, M1 HOLE M3, M2 HOLE M3, M3 HOLE, M4 HOLE, U1 LTV-357T, U2 LTV-357T, U3 LTV-357T, U4 LTV-357T, U5 LTV-357T, U6 LTV-357T, U7 LTV-357T

Commit message: Interview task submission
Routing:
- net GND: track 0.00 -> 157.2 mm
- net Earth: track 0.00 -> 154.6 mm
- net GND_Permanent: track 0.00 -> 134.7 mm
- net GND_Switched: track 0.00 -> 100.3 mm, vias 0 -> 2
- net Net-(F3-Pad1): track 0.00 -> 70.9 mm, vias 0 -> 5
- net Reversing_Signal: track 0.00 -> 56.8 mm, vias 0 -> 1
- net Reversing_Lamps: track 0.00 -> 53.4 mm
- net 12V_Switched: track 0.00 -> 50.5 mm, vias 0 -> 1
- net Net-(F1-Pad1): track 0.00 -> 50.2 mm, vias 0 -> 3
- net Tail_Lamps_Left_Signal: track 0.00 -> 45.7 mm, vias 0 -> 1
- net Tail_Lamps_Left: track 0.00 -> 44.8 mm, vias 0 -> 1
- net 12V_Permanent: track 0.00 -> 44.6 mm, vias 0 -> 1
- net Left_Turn_Signal_Lamp: track 0.00 -> 41.8 mm, vias 0 -> 1
- net Stop_Lamps: track 0.00 -> 40.8 mm, vias 0 -> 1
- net Stop_Signal: track 0.00 -> 39.2 mm, vias 0 -> 1
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