File: hw/sch_pcb/ISO11446PWR01.kicad_sch (KiCad schematic)
At the start: 8 parts, among them J1 Umin ... Umax, M1 HOLE M3, M2 HOLE M3, M3 HOLE, M4 HOLE

Commit message: testing schema
Parts:
- added F1: Fuse, Fuse:Fuse_Bourns_MF-RG400, symbol Device:Fuse
- added F2: Polyfuse, Fuse:Fuse_Bourns_MF-RG400, symbol Device:Polyfuse
- added J1, J2, J3: HEADER_2x04_PARALLEL, Mlab_Pin_Headers:Straight_2x04, symbol MLAB_HEADER:HEADER_2x04_PARALLEL
- added J4, J5, J6, J7: Conn_01x01_Female, Mlab_CON:WAGO256, symbol Connector:Conn_01x01_Female
- renumbered J1 to J8
Connections:
- net GND: no longer M1.1, M2.1, M3.1, M4.1
- new net: M1.1, M2.1, M3.1, M4.1
- new net: J1.3, J1.4, J6.1 (Pin_1)
- new net: J2.1, J2.2
- new net: J2.3, J2.4
- new net: F1.1, J1.7, J1.8, J2.5, J2.6, J2.7, J2.8
- new net: F1.2, J4.1 (Pin_1)
- new net: J1.1, J1.2, J3.7, J3.8, J7.1 (Pin_1)
- new net: F2.1, J1.5, J1.6
- new net: J3.1, J3.2
- new net: J3.3, J3.4
- new net: J3.5, J3.6
- new net: F2.2, J5.1 (Pin_1)
- no-connect marks 0 -> 5
Other:
- title: NAME -> ISO11446PWR01
